File: pcb/c64-megacart.kicad_pcb (KiCad board)
At the start: 2 copper layers, 58.4 x 50.8 mm, 12 parts, among them J1 Jumper, J2 A13switch, SW1 RESET, SW2 SW_DIP_x08, U1 C64-Exp-Port, U2 SST39SF040

Commit message: Changing design
Parts:
- removed the G*** at (62.9, 56.9)
- added G001: LOGO, components:puni, F.Cu at (63.8, 55.3)
- moved G*** 3.26 mm to (59.7, 44.6), turned to 45 degrees
Other:
- board text added: "8k"
- board text removed: "64x8kb cartridge"
- board text removed: "switch"
