File: pcb/c64-megacart.kicad_sch (KiCad schematic)
At the start: 10 parts, among them J1 Jumper, J2 A13switch, SW1 RESET, SW2 SW_DIP_x08, U1 C64-Exp-Port, U2 SST39SF040

Commit message: Changing design
Other:
- title: (none) -> C64 MegaCartridge
Changed lines of the file:
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@@
 	(paper "A4")
 	(title_block
-		(date "2021-08-15")
+		(title "C64 MegaCartridge")
+		(date "2024-08-28")
 	)
 	(junction
